File: hardware/cardboard-bot.kicad_sch (KiCad schematic)
At the start: 95 parts, among them J1 USB-C CHARGE, J10 ESC PWR 2, J2 I2C, J3 MOTOR L, J4 MOTOR R, J5 OUT1, J6 OUT2, J7 IO3, J8 IO21, J9 ESC PWR 1, Q1 CJAC80N03 DSG, Q2 CJAC80N03 CHG, Q3 AGM30P05A, SW1 POWER, U1 BQ25887RGER, U2 HY2120-CB, U3 TPS563201DDCR, U4 XIAO ESP32-C3, U5 DRV8833PWPR, U6 74VHCT1G125

Commit message: Rework BOM for JLC stock: IP2320 charger, Basic parts, no shortfalls
Swap every out-of-stock or short part for a Basic, no-fee Preferred, or high-stock Extended part
(stock checked 28 Oct 2026):

- Charger: BQ25887 -> IP2320 (8.40 V / 1.0 A straps), plus 2x HY2213-BB3A cell balancers
  with AO3401A + 100R bleed
- Buck: TPS563201 (out of stock) -> TPS54202, same SOT-23-6 pinout, 75k/10k feedback
- Status LED: WS2812B-B (out of stock) -> XL-5050RGBC-2812B-S, run through a 1N4148W from 5 V;
  the 74VHCT1G125 level shifter is removed
- FETs: HYG015N03LS1C2 for the BMS, CJAB35P03 for the power switch
- Surge diode: SMAJ10A (Preferred)
- DRV8833 sense resistors: 0.1R Basic (2 A limit)
- Bulk electrolytics: through-hole, hand-soldered; the 220 uF on VSYS is dropped
- Battery sense: VSYS/4 on GPIO3 through cuttable jumper JP1

Re-placed and re-routed the charger and balancer area. DRC: no clearance errors,
no unconnected items; a new gnd_check.py confirms one GND cluster.
BOM: 35 lines, 12 Extended (was 18), about $6.40 of parts per board.
Parts:
- removed C12: 220uF 16V, Capacitor_SMD:CP_Elec_6.3x7.7, symbol Device:C_Polarized
- removed C29: 100nF, Capacitor_SMD:C_0603_1608Metric, symbol Device:C
- removed C5: 4.7uF, Capacitor_SMD:C_0603_1608Metric, symbol Device:C
- removed C6, C7: 22uF, Capacitor_SMD:C_0805_2012Metric, symbol Device:C
- removed C8, C9: 10uF, Capacitor_SMD:C_0805_2012Metric, symbol Device:C
- removed R3: 22R 1W, Resistor_SMD:R_2512_6332Metric, symbol Device:R
- removed R5: 5.1k, Resistor_SMD:R_0603_1608Metric, symbol Device:R
- removed R6: 30k, Resistor_SMD:R_0603_1608Metric, symbol Device:R
- removed U1: BQ25887RGER, Package_DFN_QFN:VQFN-24-1EP_4x4mm_P0.5mm_EP2.5x2.5mm, symbol Battery_Management:BQ25887
- removed U3: TPS563201DDCR, Package_TO_SOT_SMD:TSOT-23-6, symbol Regulator_Switching:TPS563200
- removed U6: 74VHCT1G125, Package_TO_SOT_SMD:SOT-353_SC-70-5, symbol 74xGxx:74LVC1G125
- added C31, C32, C33: 100nF, Capacitor_SMD:C_0603_1608Metric, symbol Device:C
- added D10: 1N4148W, Diode_SMD:D_SOD-123, symbol Device:D
- added JP1: VBAT>IO3, Jumper:SolderJumper-2_P1.3mm_Bridged_RoundedPad1.0x1.5mm, symbol Jumper:SolderJumper_2_Bridged
- added Q4, Q5: AO3401A, Package_TO_SOT_SMD:SOT-23, symbol Device:Q_PMOS_GSD
- added R27: 300k, Resistor_SMD:R_0603_1608Metric, symbol Device:R
- added R28: 100k, Resistor_SMD:R_0603_1608Metric, symbol Device:R
- added R29, R31: 330R, Resistor_SMD:R_0603_1608Metric, symbol Device:R
- added R30, R32: 100R, Resistor_SMD:R_1206_3216Metric, symbol Device:R
- added U1: IP2320, Package_SO:SOIC-8-1EP_3.9x4.9mm_P1.27mm_EP2.41x3.3mm, symbol cgw:IP2320
- added U3: TPS54202DDCR, Package_TO_SOT_SMD:TSOT-23-6, symbol Regulator_Switching:TPS54202DDC
- added U7, U8: HY2213-BB3A, Package_TO_SOT_SMD:SOT-23-6, symbol cgw:HY2213
- C1: value 1uF -> 22uF; footprint Capacitor_SMD:C_0603_1608Metric -> Capacitor_SMD:C_0805_2012Metric; LCSC C15849 -> C45783; MPN CL10A105KB8NNNC -> CL21A226MAQNNNE
- C13, C27: footprint Capacitor_SMD:CP_Elec_8x10 -> Capacitor_THT:CP_Radial_D8.0mm_P3.50mm; Assembly jlc -> hand; LCSC C82006 -> (none); MPN RVT1C471M0810 -> 470uF 16V radial, 8 mm dia, 3.5 mm pitch, low ESR
- C19: footprint Capacitor_SMD:CP_Elec_6.3x7.7 -> Capacitor_THT:CP_Radial_D6.3mm_P2.50mm; Assembly jlc -> hand; LCSC C179798 -> (none); MPN 16CE220AX -> 220uF 16V radial, 6.3 mm dia, 2.5 mm pitch
- C2: value 10uF -> 22uF; LCSC C15850 -> C45783; MPN CL21A106KAYNNNE -> CL21A226MAQNNNE
- C4: value 47nF -> 100nF; LCSC C1622 -> C14663; MPN CL10B473KB8NNNC -> CC0603KRX7R9BB104
- D1: value YELLOW -> RED; LCSC C72038 -> C2286; MPN 0603 yellow LED (JLC basic, colour to confirm) -> KT-0603R
- D2: value SMBJ9.0A -> SMAJ10A; footprint Diode_SMD:D_SMB -> Diode_SMD:D_SMA; LCSC C3720683 -> C41376407; MPN SMBJ9.0A -> SMAJ10A
- D9: value WS2812B -> XL-5050RGBC-2812B-S; LCSC C2761795 -> C22461793; MPN WS2812B-B/T -> XL-5050RGBC-2812B-S
- L1: value 1uH 4A -> 2.2uH 4.8A; LCSC C5291823 -> C602029; MPN CKCS4030-1uH/N -> FHD4020S-2R2MT
- L2: value 4.7uH 2A -> 10uH 2.35A; LCSC C354587 -> C602032; MPN CKCS4030-4.7uH/M -> FHD4020S-100MT
- Q1: value CJAC80N03 DSG -> HYG015N03LS1C2 DSG; LCSC C504096 -> C18222234; MPN CJAC80N03 -> HYG015N03LS1C2
- Q2: value CJAC80N03 CHG -> HYG015N03LS1C2 CHG; LCSC C504096 -> C18222234; MPN CJAC80N03 -> HYG015N03LS1C2
- Q3: value AGM30P05A -> CJAB35P03; footprint Package_DFN_QFN:PQFN-8-EP_6x5mm_P1.27mm_Generic -> Package_SO:Vishay_PowerPAK_1212-8_Single; LCSC C6719407 -> C504071; MPN AGM30P05A -> CJAB35P03
- R13: value 56k -> 75k; LCSC C23206 -> C23242; MPN 0603WAF5602T5E -> 0603WAF7502T5E
- R18, R19: value 0.15R -> 0.1R; LCSC C104932 -> C25334; MPN RTT06R150FTP -> 1206W4F100LT5E
- R7: value 2.2k -> 1k; LCSC C4190 -> C21190; MPN 0603WAF2201T5E -> 0603WAF1001T5E
- TH1: value 10k B3950 -> 10k B3380; LCSC C47118797 -> C13564; MPN CMFA103F3950HANT -> NCP18XH103F03RB
Connections:
- net CHG_STAT is gone; now on net GND: D1.1 (K)
- net LED_DIN5 is gone; now on net LED_DIN3: R26.1
- net +5V: now also D10.2 (A); no longer C30.1, D9.1 (VDD)
- net BAT+: now also C3.1, Q4.2 (S), R29.1, U1.2 (VOUT)
- net BUCK_BST: now also U3.6 (BOOT)
- net BUCK_FB: now also U3.4 (FB)
- net BUCK_SW: now also U3.2 (SW)
- net B_NEG: now also C33.2, R32.2, U8.3 (VSS)
- net GND: now also C31.2, R28.2, U1.9 (GND), U3.1 (GND)
- net IO3: now also JP1.2 (B)
- net MID: now also C32.2, Q5.2 (S), R30.2, R31.1, U7.3 (VSS)
- net VBUS: now also L1.1, U1.6 (VIN)
- net VHOLD: now also U3.3 (VIN)
- net VSYS: now also R27.1
- net CHG_BTST renamed CHG_BST
- net CHG_BST: now also U1.7 (BST)
- net CHG_LED_A renamed PWR_LED_A
- net CHG_SW renamed CHG_LX
- net CHG_LX: now also U1.8 (LX)
- net CHG_TS renamed CHG_NTC
- net CHG_NTC: now also U1.4 (NTC)
- removed net PMID: C2.1, C3.1, L1.1
- new net BAL1_D: Q4.3 (D), R30.1
- new net BAL1_G: Q4.1 (G), U7.6 (OUT)
- new net BAL1_VDD: C32.1, R29.2, U7.2 (VDD)
- new net BAL2_D: Q5.3 (D), R32.1
- new net BAL2_G: Q5.1 (G), U8.6 (OUT)
- new net BAL2_VDD: C33.1, R31.2, U8.2 (VDD)
- new net CHG_VSYS: C2.1, U1.1 (VSYS)
- new net LED_VDD: C30.1, D10.1 (K), D9.1 (VDD)
- new net VBAT_SNS: C31.1, JP1.1 (A), R27.2, R28.1
- no-connect marks 11 -> 18
Other:
- note added: "1 USB-C charge input + IP2320 2S boost charger"
- note added: "2b Cell balancing (2x HY2213)"
- note added: "4 Hold-up + 5 V buck (TPS54202), XIAO feed"
- note added: "5 XIAO ESP32-C3, I2C, battery sense"
- note added: "6 DRV8833 drive, 2 A current limit"
- note added: "Battery sense: VSYS/4 on GPIO3 through bridged jumper JP1 (cut JP1 to use IO3 as plain GPIO)."
- note added: "Confirm before ordering: IP2320 typical application (VSET/ISET straps, VSYS/VOUT/VIN caps), HY2213 pinout + bleed circuit, HY2120 RC values."
- note removed: "1 USB-C charge input + BQ25887 2S balance charger"
- note removed: "4 Hold-up + 5 V buck (TPS563201), XIAO feed"
- note removed: "5 XIAO ESP32-C3, I2C"
- note removed: "6 DRV8833 drive, 1.3 A current limit"
- note removed: "Values to confirm against datasheets before ordering: BQ25887 caps (SNS 44uF, PMID, REGN, BTST), L1, CBSET R3, TS divider, HY2120 RC values."

Commit message: Rev A: apply datasheet checks, re-layout around real 18650 clip footprint
- MY-18650-01 clip footprint per drawing (3 legs, 1.8 mm holes, 48 mm per cell);
  cells, BMS, balancers and charger re-placed, board re-routed, DRC clean
- IP2320 wired per typical application: VIN RC + 5.1k, VSET/NTC caps,
  charge LED on LED/ISET
- HY2213 VDD resistor 100R
- Regenerated gerbers, BOM, CPL, BOM check and previews
Parts:
- added C5: 10uF, Capacitor_SMD:C_0805_2012Metric, symbol Device:C
- added C6, C7: 100nF, Capacitor_SMD:C_0603_1608Metric, symbol Device:C
- added R3: 5.1k, Resistor_SMD:R_0603_1608Metric, symbol Device:R
- added R4: 1R, Resistor_SMD:R_0603_1608Metric, symbol Device:R
- R29, R31: value 330R -> 100R; LCSC C23138 -> C22775; MPN 0603WAF3300T5E -> 0603WAF1000T5E
- U1: footprint Package_SO:SOIC-8-1EP_3.9x4.9mm_P1.27mm_EP2.41x3.3mm -> Package_SO:SOIC-8-1EP_3.9x4.9mm_P1.27mm_EP2.29x3mm
Connections:
- net CHG_NTC: now also C7.1
- net GND: now also C5.2, C6.2, C7.2, R3.2
- net VBUS: now also R3.1, R4.1; no longer R7.1, U1.6 (VIN)
- net CHG_VSET: now reaches U1.3 (VSET)
- net CHG_VSET: now also C6.1
- net CHG_LED: now reaches U1.5 (LED/ISET)
- net CHG_LED: now also R7.1
- net PWR_LED_A renamed CHG_LED_A
- new net CHG_VIN: C5.1, R4.2, U1.6 (VIN)
- no-connect marks 18 -> 16
Other:
- note added: "IP2320 per INJOINIC V1.00 datasheet fig. 5; HY2213 per HYCON DS-HY2213-V05 P-MOSFET example; clip per MYOUNG WD-CP-0056."
- note removed: "Confirm before ordering: IP2320 typical application (VSET/ISET straps, VSYS/VOUT/VIN caps), HY2213 pinout + bleed circuit, HY2120 RC values."

Commit message: Simplify rev A: off-board power switch, no balancing, LED strip pads
- SW1: 18 AWG wire pads for a 10 A+ panel switch; Q3, R11, R12 and the slide switch removed
- Cell balancers (U7, U8, Q4, Q5, R29-R32, C32, C33) removed; BMS still cuts at 4.28 V
- NTC replaced by a fixed 10k (R33); NTC fits the same pads
- D2: SMF10CA (Preferred) instead of SMAJ10A
- C1, C20: 10 uF instead of 22 uF
- J11: pads for one LED cut from a WS2812B strip; TP4 removed
- Re-routed, DRC clean; new gerbers, BOM, CPL, previews
Parts:
- removed C32, C33: 100nF, Capacitor_SMD:C_0603_1608Metric, symbol Device:C
- removed D2: SMAJ10A, Diode_SMD:D_SMA, symbol Device:D_Zener
- removed D9: XL-5050RGBC-2812B-S, LED_SMD:LED_WS2812B_PLCC4_5.0x5.0mm_P3.2mm, symbol LED:WS2812B
- removed Q3: CJAB35P03, Package_SO:Vishay_PowerPAK_1212-8_Single, symbol cgw:PMOS_PDFN
- removed Q4, Q5: AO3401A, Package_TO_SOT_SMD:SOT-23, symbol Device:Q_PMOS_GSD
- removed R11: 100k, Resistor_SMD:R_0603_1608Metric, symbol Device:R
- removed R12: 10k, Resistor_SMD:R_0603_1608Metric, symbol Device:R
- removed R29, R31: 100R, Resistor_SMD:R_0603_1608Metric, symbol Device:R
- removed R30, R32: 100R, Resistor_SMD:R_1206_3216Metric, symbol Device:R
- removed SW1: POWER, Button_Switch_THT:SW_Slide_SPDT_Straight_CK_OS102011MS2Q, symbol Switch:SW_SPDT
- removed TH1: 10k B3380, Resistor_SMD:R_0603_1608Metric, symbol Device:Thermistor_NTC
- removed TP4: +5V, TestPoint:TestPoint_Pad_D1.5mm, symbol Connector:TestPoint
- removed U7, U8: HY2213-BB3A, Package_TO_SOT_SMD:SOT-23-6, symbol cgw:HY2213
- added D2: SMF10CA, Diode_SMD:D_SOD-123F, symbol Device:D_TVS
- added J11: LED STRIP, cgw:WS2812B_Strip_1LED, symbol Connector_Generic:Conn_01x03
- added R33: 10k, Resistor_SMD:R_0603_1608Metric, symbol Device:R
- added SW1: POWER SW, Connector_Wire:SolderWire-1sqmm_1x02_P5.4mm_D1.4mm_OD2.7mm, symbol Switch:SW_SPST
- C1, C20: value 22uF -> 10uF; LCSC C45783 -> C15850; MPN CL21A226MAQNNNE -> CL21A106KAYNNNE
Connections:
- net CHG_NTC: now also R33.1
- net GND: now also D2.2 (A2), J11.3 (Pin_3), R33.2
- net LED_DIN: now also J11.2 (Pin_2)
- net LED_VDD: now also J11.1 (Pin_1)
- net VFUSE: now also SW1.1 (A)
- net VSYS: now also D2.1 (A1), SW1.2 (B)
- no-connect marks 16 -> 8
Other:
- note added: "3 Power switch (off-board), surge clamp, bulk"
- note added: "8 RGB status LED (WS2812B strip piece)"
- note removed: "2b Cell balancing (2x HY2213)"
- note removed: "3 Power switch (P-FET), surge clamp, bulk"
- note removed: "8 RGB status LED"

Commit message: Rev B board: 2S/3S LiPo on a screw terminal, two DRV8870s, smaller
- Removed the 18650 clips, USB-C charger and BMS; battery comes in on a 5.08 mm
  screw terminal, then the 20 A fuse and the switch pads
- Everything on the battery rail rated above 3S: two DRV8870 drivers (45 V, 2.5 A limit),
  SMAJ13A clamp, 25 V bulk capacitors; battery sense is now pack / 6
- 10k pull-downs on all four motor inputs and all three outputs
- Motor terminals on opposite edges (LEFT MOTOR / RIGHT MOTOR), ESC power on the right
- 60 x 46 mm (was 80 x 46), nothing on the back; 20 BOM lines, 3 Extended
- Routed, DRC clean; new gerbers, BOM, CPL, schematic, previews and docs
Parts:
- removed BT1, BT2, BT3, BT4: 18650 clip, cgw:Clip_MY-18650-01, symbol cgw:BattClip
- removed C1, C20, C23: 10uF, Capacitor_SMD:C_0805_2012Metric, symbol Device:C
- removed C13, C27: 470uF 16V, Capacitor_THT:CP_Radial_D8.0mm_P3.50mm, symbol Device:C_Polarized
- removed C19: 220uF 16V, Capacitor_THT:CP_Radial_D6.3mm_P2.50mm, symbol Device:C_Polarized
- removed C2: 22uF, Capacitor_SMD:C_0805_2012Metric, symbol Device:C
- removed C21, C22, C24, C30, C31: 100nF, Capacitor_SMD:C_0603_1608Metric, symbol Device:C
- removed C25: 2.2uF, Capacitor_SMD:C_0402_1005Metric, symbol Device:C
- removed C26: 10nF, Capacitor_SMD:C_0402_1005Metric, symbol Device:C
- removed D1: RED, LED_SMD:LED_0603_1608Metric, symbol Device:LED
- removed D10: 1N4148W, Diode_SMD:D_SOD-123, symbol Device:D
- removed D2: SMF10CA, Diode_SMD:D_SOD-123F, symbol Device:D_TVS
- removed D7, D8: 1N5819WS, Diode_SMD:D_SOD-323, symbol Device:D_Schottky
- removed J1: USB-C CHARGE, Connector_USB:USB_C_Receptacle_HRO_TYPE-C-31-M-12, symbol Connector:USB_C_Receptacle_USB2.0_16P
- removed J10: ESC PWR 2, TerminalBlock_Phoenix:TerminalBlock_Phoenix_MKDS-1,5-2-5.08_1x02_P5.08mm_Horizontal, symbol Connector_Generic:Conn_01x02
- removed J11: LED STRIP, cgw:WS2812B_Strip_1LED, symbol Connector_Generic:Conn_01x03
- removed J8: IO21, Connector_PinHeader_2.54mm:PinHeader_1x03_P2.54mm_Vertical, symbol Connector_Generic:Conn_01x03
- removed JP1: VBAT>IO3, Jumper:SolderJumper-2_P1.3mm_Bridged_RoundedPad1.0x1.5mm, symbol Jumper:SolderJumper_2_Bridged
- removed L2: 10uH 2.35A, Inductor_SMD:L_Cenker_CKCS4030, symbol Device:L
- removed Q1: HYG015N03LS1C2 DSG, Package_DFN_QFN:PQFN-8-EP_6x5mm_P1.27mm_Generic, symbol cgw:NMOS_PDFN
- removed Q2: HYG015N03LS1C2 CHG, Package_DFN_QFN:PQFN-8-EP_6x5mm_P1.27mm_Generic, symbol cgw:NMOS_PDFN
- removed R22: 1k, Resistor_SMD:R_0603_1608Metric, symbol Device:R
- removed R23, R33: 10k, Resistor_SMD:R_0603_1608Metric, symbol Device:R
- removed R24, R25, R26: 330R, Resistor_SMD:R_0603_1608Metric, symbol Device:R
- removed R27: 300k, Resistor_SMD:R_0603_1608Metric, symbol Device:R
- removed R28: 100k, Resistor_SMD:R_0603_1608Metric, symbol Device:R
- removed TP5: +3V3, TestPoint:TestPoint_Pad_D1.5mm, symbol Connector:TestPoint
- removed TP6: GND, TestPoint:TestPoint_Pad_D1.5mm, symbol Connector:TestPoint
- removed TP7: MID, TestPoint:TestPoint_Pad_D1.5mm, symbol Connector:TestPoint
- removed U1: IP2320, Package_SO:SOIC-8-1EP_3.9x4.9mm_P1.27mm_EP2.29x3mm, symbol cgw:IP2320
- removed U2: HY2120-CB, Package_TO_SOT_SMD:SOT-23-6, symbol cgw:HY2120
- removed U3: TPS54202DDCR, Package_TO_SOT_SMD:TSOT-23-6, symbol Regulator_Switching:TPS54202DDC
- removed U4: XIAO ESP32-C3, cgw:XIAO_Socket, symbol cgw:XIAO_ESP32C3
- removed U5: DRV8833PWPR, Package_SO:HTSSOP-16-1EP_4.4x5mm_P0.65mm_EP3.4x5mm_Mask2.46x2.31mm, symbol Driver_Motor:DRV8833PWP
- added C1, C2: 470uF 25V, Capacitor_THT:CP_Radial_D8.0mm_P3.50mm, symbol Device:C_Polarized
- added C12, C13: 100nF, Capacitor_SMD:C_0603_1608Metric, symbol Device:C
- added C9: 10uF, Capacitor_SMD:C_0805_2012Metric, symbol Device:C
- added D1: SMAJ13A, Diode_SMD:D_SMA, symbol Device:D_Zener
- added D2: SS34, Diode_SMD:D_SMA, symbol Device:D_Schottky
- added D7: 1N4148W, Diode_SMD:D_SOD-123, symbol Device:D
- added J1: BATTERY, TerminalBlock_Phoenix:TerminalBlock_Phoenix_MKDS-1,5-2-5.08_1x02_P5.08mm_Horizontal, symbol Connector_Generic:Conn_01x02
- added J10: LED STRIP, cgw:WS2812B_Strip_1LED, symbol Connector_Generic:Conn_01x03
- added J8: ESC PWR 1, TerminalBlock_Phoenix:TerminalBlock_Phoenix_MKDS-1,5-2-5.08_1x02_P5.08mm_Horizontal, symbol Connector_Generic:Conn_01x02
- added R11, R12: 10k, Resistor_SMD:R_0603_1608Metric, symbol Device:R
- added R5: 100k, Resistor_SMD:R_0603_1608Metric, symbol Device:R
- added R6: 20k, Resistor_SMD:R_0603_1608Metric, symbol Device:R
- added TP1: +3V3, TestPoint:TestPoint_Pad_D1.5mm, symbol Connector:TestPoint
- added TP2: GND, TestPoint:TestPoint_Pad_D1.5mm, symbol Connector:TestPoint
- added U1: TPS54202DDCR, Package_TO_SOT_SMD:TSOT-23-6, symbol Regulator_Switching:TPS54202DDC
- added U2: XIAO ESP32-C3, cgw:XIAO_Socket, symbol cgw:XIAO_ESP32C3
- added U3, U4: DRV8870DDAR, Package_SO:Texas_HTSOP-8-1EP_3.9x4.9mm_P1.27mm_EP2.95x4.9mm_Mask2.4x3.1mm_ThermalVias, symbol Driver_Motor:DRV8870DDA
- C16: value 100nF -> 10uF; footprint Capacitor_SMD:C_0603_1608Metric -> Capacitor_SMD:C_0805_2012Metric; LCSC C14663 -> C15850; MPN CC0603KRX7R9BB104 -> CL21A106KAYNNNE
- C17, C18: value 22uF -> 100nF; footprint Capacitor_SMD:C_0805_2012Metric -> Capacitor_SMD:C_0603_1608Metric; LCSC C45783 -> C14663; MPN CL21A226MAQNNNE -> CC0603KRX7R9BB104
- C5: value 10uF -> 100nF; footprint Capacitor_SMD:C_0805_2012Metric -> Capacitor_SMD:C_0603_1608Metric; LCSC C15850 -> C14663; MPN CL21A106KAYNNNE -> CC0603KRX7R9BB104
- C6, C7: value 100nF -> 22uF; footprint Capacitor_SMD:C_0603_1608Metric -> Capacitor_SMD:C_0805_2012Metric; LCSC C14663 -> C45783; MPN CC0603KRX7R9BB104 -> CL21A226MAQNNNE
- D3: value SS34 -> B5819W; footprint Diode_SMD:D_SMA -> Diode_SMD:D_SOD-123; LCSC C8678 -> C8598; MPN SS34 -> B5819W SL
- D4: value B5819W -> 1N5819WS; footprint Diode_SMD:D_SOD-123 -> Diode_SMD:D_SOD-323; LCSC C8598 -> C191023; MPN B5819W SL -> 1N5819WS
- J3: value MOTOR L -> LEFT MOTOR
- J4: value MOTOR R -> RIGHT MOTOR
- J7: value IO3 -> OUT3
- J9: value ESC PWR 1 -> ESC PWR 2
- L1: value 2.2uH 4.8A -> 10uH 2.35A; LCSC C602029 -> C602032; MPN FHD4020S-2R2MT -> FHD4020S-100MT
- R1: value 5.1k -> 75k; LCSC C23186 -> C23242; MPN 0603WAF5101T5E -> 0603WAF7502T5E
- R10: value 2k -> 33k; LCSC C22975 -> C4216; MPN 0603WAF2001T5E -> 0603WAF3302T5E
- R13: value 75k -> 10k; LCSC C23242 -> C25804; MPN 0603WAF7502T5E -> 0603WAF1002T5E
- R15, R16: value 4.7k -> 1k; LCSC C23162 -> C21190; MPN 0603WAF4701T5E -> 0603WAF1001T5E
- R17: value 10k -> 1k; LCSC C25804 -> C21190; MPN 0603WAF1002T5E -> 0603WAF1001T5E
- R18, R19: value 0.1R -> 10k; footprint Resistor_SMD:R_1206_3216Metric -> Resistor_SMD:R_0603_1608Metric; LCSC C25334 -> C25804; MPN 1206W4F100LT5E -> 0603WAF1002T5E
- R2: value 5.1k -> 10k; LCSC C23186 -> C25804; MPN 0603WAF5101T5E -> 0603WAF1002T5E
- R20, R9: value 1k -> 10k; LCSC C21190 -> C25804; MPN 0603WAF1001T5E -> 0603WAF1002T5E
- R21: value 10k -> 330R; LCSC C25804 -> C23138; MPN 0603WAF1002T5E -> 0603WAF3300T5E
- R3: value 5.1k -> 4.7k; LCSC C23186 -> C23162; MPN 0603WAF5101T5E -> 0603WAF4701T5E
- R4: value 1R -> 4.7k; LCSC C22936 -> C23162; MPN 0603WAF100KT5E -> 0603WAF4701T5E
- R7: value 1k -> 0.1R; footprint Resistor_SMD:R_0603_1608Metric -> Resistor_SMD:R_1206_3216Metric; LCSC C21190 -> C25334; MPN 0603WAF1001T5E -> 1206W4F100LT5E
- R8: value 330R -> 0.1R; footprint Resistor_SMD:R_0603_1608Metric -> Resistor_SMD:R_1206_3216Metric; LCSC C23138 -> C25334; MPN 0603WAF3300T5E -> 1206W4F100LT5E
- SW1: footprint Connector_Wire:SolderWire-1sqmm_1x02_P5.4mm_D1.4mm_OD2.7mm -> Connector_Wire:SolderWire-0.75sqmm_1x02_P4.8mm_D1.25mm_OD2.3mm; MPN SPST rocker or toggle, 10 A+ at 12 V DC, panel mount, 18 AW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 -> SPST rocker or toggle, 10 A+ at 16 V DC, panel mount, 18 AW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
Connections:
- net BMS_CS is gone; now on net GND: R10.2
- net B_NEG is gone; now on net GND: C10.2, C11.2
- net CC1 is gone; now on net +5V: R1.1
- net CC2 is gone; now on net BUCK_FB: R2.1
- net CHG_BST is gone; now on net VHOLD: C4.1
- net CHG_LED_A is gone; now on net GND: R7.2
- net CHG_NTC is gone; now on net +5V: C7.1
- net CHG_VSET is gone; now on net +5V: C6.1
- net DRV_AISEN is gone; now on net IO10: R18.1
- net DRV_BISEN is gone; now on net IO20: R19.1
- net IO3_SIG is gone; now on net OUT3_SIG: J7.3 (Pin_3)
- net MID is gone; now on net +3V3: R9.1
- net +3V3: now also C11.1, R3.1, R4.1, TP1.1, U2.12 (3V3); no longer R15.1, R16.1
- net +5V: now also D3.2 (A), L1.2, D7.2 (A); no longer C17.1, C18.1, R13.1, R17.1
- net +5V_XIAO: now also C10.1, D3.1 (K), C9.1, U2.14 (5V); no longer D4.1 (K)
- net AIN1: now also R11.1, U2.3 (D2/GPIO4), U3.3 (IN1)
- net AIN2: now also R12.1, U2.4 (D3/GPIO5), U3.2 (IN2)
- net BAT+: now also J1.1 (Pin_1); no longer C3.1, R8.1
- net BIN1: now also R13.1, U2.5 (D4/GPIO6), U4.3 (IN1)
- net BIN2: now also R14.1, U2.6 (D5/GPIO7), U4.2 (IN2)
- net BUCK_BST: now also C5.1, U1.6 (BOOT); no longer C16.1
- net BUCK_FB: now also R1.2, U1.4 (FB); no longer R13.2, R14.1
- net BUCK_SW: now also C5.2, L1.1, U1.2 (SW); no longer C16.2
- net GND: now also C16.2, C4.2, R13.2, R20.2, R8.2, C1.2, C12.2, C13.2, C2.2, C9.2, D1.2 (A), J1.2 (Pin_2), J10.3 (Pin_3), J8.2 (Pin_2), R11.2, R12.2, R6.2, TP2.1, U1.1 (GND), U2.13 (GND), U3.1 (GND), U3.9 (GND), U4.1 (GND), U4.9 (GND); no longer C5.2, R1.2, R10.1, R21.2, R3.2
- net IO10: now also R15.1, U2.11 (D10/GPIO10); no longer R20.1, R21.1
- net IO20: now also R16.1, U2.8 (D7/GPIO20)
- net IO21: now also R17.1, R20.1, U2.7 (D6/GPIO21)
- net LED_DIN: now also R21.2, J10.2 (Pin_2)
- net LED_DIN3: now also R21.1, U2.10 (D9/GPIO9)
- net LED_VDD: now also C18.1, D7.1 (K), J10.1 (Pin_1)
- net MOTL_A: now also U3.6 (OUT1)
- net MOTL_B: now also U3.8 (OUT2)
- net MOTR_A: now also U4.6 (OUT1)
- net MOTR_B: now also U4.8 (OUT2)
- net OUT1_SIG: now also R15.2; no longer R20.2
- net OUT1_VP: now also D4.1 (K); no longer D5.1 (K)
- net OUT2_SIG: now also R16.2
- net OUT2_VP: now also D5.1 (K); no longer D6.1 (K)
- net SCL: now also R4.2, U2.9 (D8/GPIO8); no longer R16.2
- net SDA: now also R3.2, U2.1 (D0/GPIO2); no longer R15.2
- net VBAT_SNS: now also C12.1, R5.2, R6.1, U2.2 (D1/GPIO3)
- net VHOLD: now also C3.1, C2.1, D2.1 (K), U1.3 (VIN); no longer C14.1, C15.1, D3.1 (K)
- net VSYS: now also C14.1, C15.1, C16.1, C17.1, C1.1, D1.1 (K), D2.2 (A), J8.1 (Pin_1), R5.1, U3.5 (VM), U4.5 (VM); no longer D3.2 (A)
- net BMS_VC renamed DRV_VREF
- net DRV_VREF: now also R10.1, C13.1, U3.4 (VREF), U4.4 (VREF); no longer C11.1
- removed net BMS_VDD: C10.1, R8.2
- net CHG_LED renamed ISEN_L
- net ISEN_L: now also U3.7 (ISEN)
- removed net CHG_LX: C4.2, L1.2
- removed net CHG_VIN: C5.1, R4.2
- net DRV_SLEEP renamed OUT3_SIG
- net IO3_VP renamed OUT3_VP
- net OUT3_VP: now also D6.1 (K)
- removed net VBUS: L1.1, R3.1, R4.1
- new net ISEN_R: R8.1, U4.7 (ISEN)
- no-connect marks 8 -> 1
Other:
- note added: "1 Battery input (2S / 3S LiPo), 20 A blade fuse, power switch, surge clamp, ESC power"
- note added: "10k pull-downs on every motor input and output keep motors and ESCs off while the ESP32 boots."
- note added: "2 Hold-up + 5 V buck (TPS54202), XIAO feed"
- note added: "3 XIAO ESP32-C3, I2C, battery sense"
- note added: "4 2x DRV8870 drive, 2.5 A current limit"
- note added: "5 PWM outputs (ESC or servo)"
- note added: "6 RGB status LED (WS2812B strip piece)"
- note added: "Cardboard Bot v2 main board - rev B - Columbia Gadget Works"
- note added: "Power: 2S or 3S LiPo on J1. Everything on VSYS is rated for 3S (12.6 V) with margin; SMAJ13A clamps spikes at about 21 V."
- note added: "XIAO pins: D0 SDA(GPIO2) D1 VBAT/6(GPIO3) D2-D3 left DRV8870 IN1/IN2 D4-D5 right DRV8870 IN1/IN2 D6 OUT3(GPIO21) D7 OUT2(GPIO20) D8 SCL(GPIO8) D9 LED(GPIO9) D10 OUT1(GPIO10)"
- note removed: "1 USB-C charge input + IP2320 2S boost charger"
- note removed: "2 Cells, 2S BMS (HY2120), 20 A blade fuse"
- note removed: "3 Power switch (off-board), surge clamp, bulk"
- note removed: "4 Hold-up + 5 V buck (TPS54202), XIAO feed"
- note removed: "5 XIAO ESP32-C3, I2C, battery sense"
- note removed: "6 DRV8833 drive, 2 A current limit"
- note removed: "7 PWM outputs (ESC or servo) + spare GPIO"
- note removed: "8 RGB status LED (WS2812B strip piece)"
- note removed: "Battery sense: VSYS/4 on GPIO3 through bridged jumper JP1 (cut JP1 to use IO3 as plain GPIO)."
- note removed: "Cardboard Bot v2 main board - rev A - Columbia Gadget Works"
- note removed: "IP2320 per INJOINIC V1.00 datasheet fig. 5; HY2213 per HYCON DS-HY2213-V05 P-MOSFET example; clip per MYOUNG WD-CP-0056."
- note removed: "XIAO pins: D0 SDA(GPIO2) D1 IO3 D2-D5 DRV8833 AIN1/AIN2/BIN1/BIN2 D6 IO21 D7 OUT2(GPIO20) D8 SCL(GPIO8) D9 LED(GPIO9) D10 OUT1(GPIO10)"
